File: hardware/peripheral/p2grv-001.brd (EAGLE design)
At the start: 18 x 31 mm, 7 parts

Commit message: Initial design.
Parts:
- moved LOGO1 0.25 mm to (2.75, 28.0), flipped to the top, turned to 0 degrees
Connections:
- net ANLG0: now also J1.2
- net ANLG1: now also J2.2
- net ANLG2: now also J3.2
- net ANLG3: now also J4.2
- net DTCT0: now also J1.1
- net DTCT1: now also J2.1
- net DTCT2: now also J3.1
- net DTCT3: now also J4.1
- net GND: now also J1.4, J2.4, J3.4, J4.4
- net VCC: now also J1.3, J2.3, J3.3, J4.3
Routing:
- net VCC: track 0.00 -> 45.2 mm
- net GND: track 0.00 -> 40.7 mm
- net ANLG3: track 0.00 -> 31.7 mm
- net ANLG2: track 0.00 -> 30.9 mm
- net ANLG0: track 0.00 -> 28.0 mm
- net DTCT0: track 0.00 -> 27.9 mm
- net DTCT3: track 0.00 -> 21.1 mm
- net DTCT1: track 0.00 -> 12.1 mm
- net ANLG1: track 0.00 -> 11.6 mm
- net DTCT2: track 0.00 -> 11.5 mm
Other:
- board text added: "GroveGear 0.0.1-X"
- board text removed: "Hex Sw 0.0.1-X"
