File: hardware/peripheral/p2grv-001.brd (EAGLE design)
At the start: 18 x 31 mm, 7 parts

Commit message: Parts number.
Parts:
- renumbered J1 to J21, J2 to J22, J3 to J23, J4 to J24
Changed lines of the file:
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@@
 </element>
 <element name="U$1" library="pineapple" package="PINEAPPLE450_SILK" value="PINEAPPLE450_SILK" x="0.5" y="21" smashed="yes" rot="MR90"/>
-<element name="J1" library="SparkFun-Connectors" library_urn="urn:adsk.eagle:library:513" package="JST-4-PTH-VERT" package3d_urn="urn:adsk.eagle:package:38102/1" value="" x="5" y="23" smashed="yes">
+<element name="J21" library="SparkFun-Connectors" library_urn="urn:adsk.eagle:library:513" package="JST-4-PTH-VERT" package3d_urn="urn:adsk.eagle:package:38102/1" value="" x="5" y="23" smashed="yes">
 <attribute name="NAME" x="5" y="24" size="1" layer="25" ratio="20" align="center"/>
 <attribute name="PROD_ID" value="CONN-13251" x="5" y="23" size="1.778" layer="27" display="off"/>
 <attribute name="VALUE" x="3.349" y="19.698" size="0.6096" layer="27" font="vector" ratio="20"/>
 </element>
-<element name="J2" library="SparkFun-Connectors" library_urn="urn:adsk.eagle:library:513" package="JST-4-PTH-VERT" package3d_urn="urn:adsk.eagle:package:38102/1" value="" x="5" y="18" smashed="yes">
+<element name="J22" library="SparkFun-Connectors" library_urn="urn:adsk.eagle:library:513" package="JST-4-PTH-VERT" package3d_urn="urn:adsk.eagle:package:38102/1" value="" x="5" y="18" smashed="yes">
 <attribute name="NAME" x="5" y="19" size="1" layer="25" ratio="20" align="center"/>
 <attribute name="PROD_ID" value="CONN-13251" x="5" y="18" size="1.778" layer="27" display="off"/>
 <attribute name="VALUE" x="3.349" y="14.698" size="0.6096" layer="27" font="vector" ratio="20"/>
 </element>
-<element name="J3" library="SparkFun-Connectors" library_urn="urn:adsk.eagle:library:513" package="JST-4-PTH-VERT" package3d_urn="urn:adsk.eagle:package:38102/1" value="" x="5" y="13" smashed="yes">
+<element name="J23" library="SparkFun-Connectors" library_urn="urn:adsk.eagle:library:513" package="JST-4-PTH-VERT" package3d_urn="urn:adsk.eagle:package:38102/1" value="" x="5" y="13" smashed="yes">
 <attribute name="NAME" x="5" y="14" size="1" layer="25" ratio="20" align="center"/>
 <attribute name="PROD_ID" value="CONN-13251" x="5" y="13" size="1.778" layer="27" display="off"/>
 <attribute name="VALUE" x="3.349" y="9.698" size="0.6096" layer="27" font="vector" ratio="20"/>
 </element>
-<element name="J4" library="SparkFun-Connectors" library_urn="urn:adsk.eagle:library:513" package="JST-4-PTH-VERT" package3d_urn="urn:adsk.eagle:package:38102/1" value="" x="5" y="8" smashed="yes">
+<element name="J24" library="SparkFun-Connectors" library_urn="urn:adsk.eagle:library:513" package="JST-4-PTH-VERT" package3d_urn="urn:adsk.eagle:package:38102/1" value="" x="5" y="8" smashed="yes">
 <attribute name="NAME" x="5" y="9" size="1" layer="25" ratio="20" align="center"/>
 <attribute name="PROD_ID" value="CONN-13251" x="5" y="8" size="1.778" layer="27" display="off"/>
@@
 <contactref element="JP1" pad="9"/>
 <contactref element="JP1" pad="13"/>
-<contactref element="J1" pad="4"/>
-<contactref element="J2" pad="4"/>
-<contactref element="J3" pad="4"/>
-<contactref element="J4" pad="4"/>
+<contactref element="J21" pad="4"/>
+<contactref element="J22" pad="4"/>
+<contactref element="J23" pad="4"/>
+<contactref element="J24" pad="4"/>
 <wire x1="8.0772" y1="22.4028" x2="8.0772" y2="17.526" width="0.1524" layer="16"/>
 <wire x1="8.0772" y1="17.526" x2="8" y2="17.45" width="0.1524" layer="16"/>
@@
 <signal name="DTCT0">
 <contactref element="JP1" pad="2"/>
-<contactref element="J1" pad="1"/>
+<contactref element="J21" pad="1"/>
 <wire x1="11.7348" y1="7.62" x2="11.7348" y2="6.7056" width="0.1524" layer="1"/>
 <wire x1="13.2588" y1="9.144" x2="11.7348" y2="7.62" width="0.1524" layer="1"/>
@@
 <contactref element="JP1" pad="12"/>
 <contactref element="JP1" pad="8"/>
-<contactref element="J1" pad="3"/>
-<contactref element="J2" pad="3"/>
-<contactref element="J3" pad="3"/>
-<contactref element="J4" pad="3"/>
+<contactref element="J21" pad="3"/>
+<contactref element="J22" pad="3"/>
+<contactref element="J23" pad="3"/>
+<contactref element="J24" pad="3"/>
 <wire x1="11.5824" y1="10.3632" x2="11.5824" y2="9.2964" width="0.1524" layer="16"/>
 <wire x1="10.668" y1="11.2776" x2="11.5824" y2="10.3632" width="0.1524" layer="16"/>
@@
 <signal name="DTCT1">
 <contactref element="JP1" pad="6"/>
-<contactref element="J2" pad="1"/>
+<contactref element="J22" pad="1"/>
 <wire x1="10.668" y1="11.7348" x2="11.5824" y2="11.7348" width="0.1524" layer="1"/>
 <wire x1="7.0104" y1="15.3924" x2="10.668" y2="11.7348" width="0.1524" layer="1"/>
@@
 <signal name="DTCT2">
 <contactref element="JP1" pad="10"/>
-<contactref element="J3" pad="1"/>
+<contactref element="J23" pad="1"/>
 <wire x1="8.8392" y1="16.764" x2="11.5824" y2="16.764" width="0.1524" layer="16"/>
 <wire x1="5.6388" y1="13.5636" x2="8.8392" y2="16.764" width="0.1524" layer="16"/>
@@
 <signal name="DTCT3">
 <contactref element="JP1" pad="14"/>
-<contactref element="J4" pad="1"/>
+<contactref element="J24" pad="1"/>
 <wire x1="11.7348" y1="20.7264" x2="11.7348" y2="21.7932" width="0.1524" layer="16"/>
 <wire x1="12.8016" y1="19.6596" x2="11.7348" y2="20.7264" width="0.1524" layer="16"/>
@@
 <signal name="ANLG0">
 <contactref element="JP1" pad="3"/>
-<contactref element="J1" pad="2"/>
+<contactref element="J21" pad="2"/>
 <wire x1="14.3256" y1="10.2108" x2="14.3256" y2="9.2964" width="0.1524" layer="16"/>
 <wire x1="15.6972" y1="11.5824" x2="14.3256" y2="10.2108" width="0.1524" layer="16"/>
@@
 <signal name="ANLG1">
 <contactref element="JP1" pad="7"/>
-<contactref element="J2" pad="2"/>
+<contactref element="J22" pad="2"/>
 <wire x1="13.1064" y1="14.3256" x2="14.1732" y2="14.3256" width="0.1524" layer="1"/>
 <wire x1="11.7348" y1="15.6972" x2="13.1064" y2="14.3256" width="0.1524" layer="1"/>
@@
 <signal name="ANLG3">
 <contactref element="JP1" pad="15"/>
-<contactref element="J4" pad="2"/>
+<contactref element="J24" pad="2"/>
 <wire x1="14.3256" y1="23.7744" x2="14.3256" y2="24.384" width="0.1524" layer="16"/>
 <wire x1="16.002" y1="22.098" x2="14.3256" y2="23.7744" width="0.1524" layer="16"/>
@@
 <signal name="ANLG2">
 <contactref element="JP1" pad="11"/>
-<contactref element="J3" pad="2"/>
+<contactref element="J23" pad="2"/>
 <wire x1="14.3256" y1="18.5928" x2="14.3256" y2="19.2024" width="0.1524" layer="1"/>
 <wire x1="15.6972" y1="17.2212" x2="14.3256" y2="18.5928" width="0.1524" layer="1"/>

Commit message: Silk.
Parts:
- moved U$1 1.00 mm to (0.50, 20.0)
Changed lines of the file:
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@@
 <setting verticaltext="up"/>
 </settings>
-<grid distance="1" unitdist="mm" unit="mm" style="lines" multiple="2" display="yes" altdistance="5" altunitdist="mil" altunit="mil"/>
+<grid distance="0.5" unitdist="mm" unit="mm" style="lines" multiple="2" display="yes" altdistance="5" altunitdist="mil" altunit="mil"/>
 <layers>
-<layer number="1" name="Top" color="4" fill="1" visible="yes" active="yes"/>
-<layer number="16" name="Bottom" color="1" fill="1" visible="yes" active="yes"/>
+<layer number="1" name="Top" color="4" fill="1" visible="no" active="yes"/>
+<layer number="16" name="Bottom" color="1" fill="1" visible="no" active="yes"/>
 <layer number="17" name="Pads" color="2" fill="1" visible="yes" active="yes"/>
 <layer number="18" name="Vias" color="2" fill="1" visible="yes" active="yes"/>
 <layer number="19" name="Unrouted" color="6" fill="1" visible="yes" active="yes"/>
 <layer number="20" name="Dimension" color="24" fill="1" visible="yes" active="yes"/>
-<layer number="21" name="tPlace" color="7" fill="1" visible="yes" active="yes"/>
-<layer number="22" name="bPlace" color="7" fill="1" visible="no" active="yes"/>
+<layer number="21" name="tPlace" color="7" fill="1" visible="no" active="yes"/>
+<layer number="22" name="bPlace" color="7" fill="1" visible="yes" active="yes"/>
 <layer number="23" name="tOrigins" color="15" fill="1" visible="yes" active="yes"/>
 <layer number="24" name="bOrigins" color="15" fill="1" visible="yes" active="yes"/>
-<layer number="25" name="tNames" color="7" fill="1" visible="yes" active="yes"/>
-<layer number="26" name="bNames" color="7" fill="1" visible="no" active="yes"/>
+<layer number="25" name="tNames" color="7" fill="1" visible="no" active="yes"/>
+<layer number="26" name="bNames" color="7" fill="1" visible="yes" active="yes"/>
 <layer number="27" name="tValues" color="7" fill="1" visible="no" active="yes"/>
 <layer number="28" name="bValues" color="7" fill="1" visible="no" active="yes"/>
@@
 <text x="8" y="5" size="1" layer="25" align="center">G</text>
 <text x="2" y="26" size="1" layer="25" align="center">0</text>
+<text x="2" y="5.5" size="1" layer="26" rot="MR0" align="center">D</text>
+<text x="4" y="5.5" size="1" layer="26" rot="MR0" align="center">A</text>
+<text x="6" y="5.5" size="1" layer="26" rot="MR0" align="center">V</text>
+<text x="8" y="5.5" size="1" layer="26" rot="MR0" align="center">G</text>
 </plain>
 <attributes>
@@
 <attribute name="VALUE" x="17.445" y="5.34" size="1.27" layer="27" rot="R90"/>
 </element>
-<element name="U$1" library="pineapple" package="PINEAPPLE450_SILK" value="PINEAPPLE450_SILK" x="0.5" y="21" smashed="yes" rot="MR90"/>
+<element name="U$1" library="pineapple" package="PINEAPPLE450_SILK" value="PINEAPPLE450_SILK" x="0.5" y="20" smashed="yes" rot="MR90"/>
 <element name="J21" library="SparkFun-Connectors" library_urn="urn:adsk.eagle:library:513" package="JST-4-PTH-VERT" package3d_urn="urn:adsk.eagle:package:38102/1" value="" x="5" y="23" smashed="yes">
 <attribute name="NAME" x="5" y="24" size="1" layer="25" ratio="20" align="center"/>

Commit message: Silk.
Parts:
- renumbered JP1 to SV1
Changed lines of the file:
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@@
 <layer number="19" name="Unrouted" color="6" fill="1" visible="yes" active="yes"/>
 <layer number="20" name="Dimension" color="24" fill="1" visible="yes" active="yes"/>
-<layer number="21" name="tPlace" color="7" fill="1" visible="no" active="yes"/>
-<layer number="22" name="bPlace" color="7" fill="1" visible="yes" active="yes"/>
+<layer number="21" name="tPlace" color="7" fill="1" visible="yes" active="yes"/>
+<layer number="22" name="bPlace" color="7" fill="1" visible="no" active="yes"/>
 <layer number="23" name="tOrigins" color="15" fill="1" visible="yes" active="yes"/>
 <layer number="24" name="bOrigins" color="15" fill="1" visible="yes" active="yes"/>
-<layer number="25" name="tNames" color="7" fill="1" visible="no" active="yes"/>
-<layer number="26" name="bNames" color="7" fill="1" visible="yes" active="yes"/>
+<layer number="25" name="tNames" color="7" fill="1" visible="yes" active="yes"/>
+<layer number="26" name="bNames" color="7" fill="1" visible="no" active="yes"/>
 <layer number="27" name="tValues" color="7" fill="1" visible="no" active="yes"/>
 <layer number="28" name="bValues" color="7" fill="1" visible="no" active="yes"/>
@@
 <elements>
 <element name="LOGO1" library="SparkFun-Aesthetics" package="OSHW-LOGO-S_COPPER" value="OSHW-LOGOS-COPPER" x="2.75" y="28" smashed="yes"/>
-<element name="JP1" library="pinhead" library_urn="urn:adsk.eagle:library:325" package="2X08" package3d_urn="urn:adsk.eagle:package:22481/2" value="" x="13" y="15.5" smashed="yes" rot="R90">
+<element name="SV1" library="pinhead" library_urn="urn:adsk.eagle:library:325" package="2X08" package3d_urn="urn:adsk.eagle:package:22481/2" value="" x="13" y="15.5" smashed="yes" rot="R90">
 <attribute name="NAME" x="17" y="6.5" size="1" layer="25" ratio="10" rot="R90" align="bottom-center"/>
 <attribute name="POPULARITY" value="6" x="13" y="15.5" size="1.778" layer="27" rot="R90" display="off"/>
@@
 <signals>
 <signal name="GND">
-<contactref element="JP1" pad="1"/>
-<contactref element="JP1" pad="5"/>
-<contactref element="JP1" pad="9"/>
-<contactref element="JP1" pad="13"/>
+<contactref element="SV1" pad="1"/>
+<contactref element="SV1" pad="5"/>
+<contactref element="SV1" pad="9"/>
+<contactref element="SV1" pad="13"/>
 <contactref element="J21" pad="4"/>
 <contactref element="J22" pad="4"/>
@@
 </signal>
 <signal name="DTCT0">
-<contactref element="JP1" pad="2"/>
+<contactref element="SV1" pad="2"/>
 <contactref element="J21" pad="1"/>
 <wire x1="11.7348" y1="7.62" x2="11.7348" y2="6.7056" width="0.1524" layer="1"/>
@@
 </signal>
 <signal name="VCC">
-<contactref element="JP1" pad="4"/>
-<contactref element="JP1" pad="16"/>
-<contactref element="JP1" pad="12"/>
-<contactref element="JP1" pad="8"/>
+<contactref element="SV1" pad="4"/>
+<contactref element="SV1" pad="16"/>
+<contactref element="SV1" pad="12"/>
+<contactref element="SV1" pad="8"/>
 <contactref element="J21" pad="3"/>
 <contactref element="J22" pad="3"/>
@@
 </signal>
 <signal name="DTCT1">
-<contactref element="JP1" pad="6"/>
+<contactref element="SV1" pad="6"/>
 <contactref element="J22" pad="1"/>
 <wire x1="10.668" y1="11.7348" x2="11.5824" y2="11.7348" width="0.1524" layer="1"/>
@@
 </signal>
 <signal name="DTCT2">
-<contactref element="JP1" pad="10"/>
+<contactref element="SV1" pad="10"/>
 <contactref element="J23" pad="1"/>
 <wire x1="8.8392" y1="16.764" x2="11.5824" y2="16.764" width="0.1524" layer="16"/>
@@
 </signal>
 <signal name="DTCT3">
-<contactref element="JP1" pad="14"/>
+<contactref element="SV1" pad="14"/>
 <contactref element="J24" pad="1"/>
 <wire x1="11.7348" y1="20.7264" x2="11.7348" y2="21.7932" width="0.1524" layer="16"/>
@@
 </signal>
 <signal name="ANLG0">
-<contactref element="JP1" pad="3"/>
+<contactref element="SV1" pad="3"/>
 <contactref element="J21" pad="2"/>
 <wire x1="14.3256" y1="10.2108" x2="14.3256" y2="9.2964" width="0.1524" layer="16"/>
@@
 </signal>
 <signal name="ANLG1">
-<contactref element="JP1" pad="7"/>
+<contactref element="SV1" pad="7"/>
 <contactref element="J22" pad="2"/>
 <wire x1="13.1064" y1="14.3256" x2="14.1732" y2="14.3256" width="0.1524" layer="1"/>
@@
 </signal>
 <signal name="ANLG3">
-<contactref element="JP1" pad="15"/>
+<contactref element="SV1" pad="15"/>
 <contactref element="J24" pad="2"/>
 <wire x1="14.3256" y1="23.7744" x2="14.3256" y2="24.384" width="0.1524" layer="16"/>
@@
 </signal>
 <signal name="ANLG2">
-<contactref element="JP1" pad="11"/>
+<contactref element="SV1" pad="11"/>
 <contactref element="J23" pad="2"/>
 <wire x1="14.3256" y1="18.5928" x2="14.3256" y2="19.2024" width="0.1524" layer="1"/>
